Commit message: Update oneleg_robot.urdf

File: udm_project/src/section_1/src/one_leg_description/src/urdf/oneleg_robot.urdf (robot description, URDF)
Before this commit: robot oneleg_robot, 3 links, 2 joints
Links:
- removed link left_h1
- removed link left_k1
- added link ball_leg_left_front; visual sphere length=0.05 radius=0.025
- added link ball_leg_left_rear; visual sphere length=0.05 radius=0.025
- added link ball_leg_right_front; visual sphere length=0.05 radius=0.025
- added link ball_leg_right_rear; visual sphere length=0.05 radius=0.025
- added link base_foot
- added link base_leg_left_front; visual cylinder length=0.05 radius=0.025
- added link base_leg_left_rear; visual cylinder length=0.05 radius=0.025
- added link base_leg_right_front; visual cylinder length=0.05 radius=0.025
- added link base_leg_right_rear; visual cylinder length=0.05 radius=0.025
- added link link_foot_leg_left_front; visual cylinder length=0.2 radius=0.02
- added link link_foot_leg_left_rear; visual cylinder length=0.2 radius=0.02
- added link link_foot_leg_right_front; visual cylinder length=0.2 radius=0.02
- added link link_foot_leg_right_rear; visual cylinder length=0.2 radius=0.02
- added link link_lower_leg_left_front; visual cylinder length=0.2 radius=0.02
- added link link_lower_leg_left_rear; visual cylinder length=0.2 radius=0.02
- added link link_lower_leg_right_front; visual cylinder length=0.2 radius=0.02
- added link link_lower_leg_right_rear; visual cylinder length=0.2 radius=0.02
- added link link_upper_leg_left_front; visual cylinder length=0.2 radius=0.03
- added link link_upper_leg_left_rear; visual cylinder length=0.2 radius=0.03
- added link link_upper_leg_right_front; visual cylinder length=0.2 radius=0.03
- added link link_upper_leg_right_rear; visual cylinder length=0.2 radius=0.03
- added link lower_leg_left_front; visual cylinder length=0.05 radius=0.025
- added link lower_leg_left_rear; visual cylinder length=0.05 radius=0.025
- added link lower_leg_right_front; visual cylinder length=0.05 radius=0.025
- added link lower_leg_right_rear; visual cylinder length=0.05 radius=0.025
- added link upper_leg_left_front; visual cylinder length=0.05 radius=0.025
- added link upper_leg_left_rear; visual cylinder length=0.05 radius=0.025
- added link upper_leg_right_front; visual cylinder length=0.05 radius=0.025
- added link upper_leg_right_rear; visual cylinder length=0.05 radius=0.025
- link base_link: mass 5 -> None; geometry visual box size=0.5 0.3 0.05
Joints:
- removed joint joint_left_h1
- removed joint joint_left_k1
- added joint ball_leg_left_front_joint: type fixed, parent link_foot_leg_left_front, child ball_leg_left_front, origin xyz=0 0.2 0  rpy=1.5707 0 0
- added joint ball_leg_left_rear_joint: type fixed, parent link_foot_leg_left_rear, child ball_leg_left_rear, origin xyz=0 0.2 0  rpy=1.5707 0 0
- added joint ball_leg_right_front_joint: type fixed, parent link_foot_leg_right_front, child ball_leg_right_front, origin xyz=0 0.2 0  rpy=1.5707 0 0
- added joint ball_leg_right_rear_joint: type fixed, parent link_foot_leg_right_rear, child ball_leg_right_rear, origin xyz=0 0.2 0  rpy=1.5707 0 0
- added joint base_link_joint: type fixed, parent base_foot, child base_link, origin xyz=0 0 0 rpy=0 0 0
- added joint joint_left_front_1: type revolute, parent base_link, child base_leg_left_front, origin xyz=0.23 0.17 0.0 rpy=1.5707 0.785 0, axis 0 0 1, limit lower=0.21 upper=1.21 effort=1000 velocity=100.0
- added joint joint_left_front_2: type revolute, parent base_leg_left_front, child link_upper_leg_left_front, origin xyz=0 0 0 rpy=1.5707 0 0, axis 1 0 0, limit lower=-0.1963 upper=0.1963 effort=1000 velocity=100.0
- added joint joint_left_front_3: type revolute, parent upper_leg_left_front, child link_lower_leg_left_front, origin xyz=0 0 0 rpy=0 1.5707 0, axis 1 0 0, limit lower=-1.64 upper=0.17 effort=1000 velocity=100.0
- added joint joint_left_front_4: type revolute, parent lower_leg_left_front, child link_foot_leg_left_front, origin xyz=0 0 0 rpy=0 1.5707 0, axis 1 0 0, limit lower=-1.63 upper=0.62 effort=1000 velocity=100.0
- added joint joint_left_rear_1: type revolute, parent base_link, child base_leg_left_rear, origin xyz=-0.23 0.17 0.0 rpy=1.5707 0.785 0, axis 0 0 1, limit lower=0.21 upper=1.21 effort=1000 velocity=100.0
- added joint joint_left_rear_2: type revolute, parent base_leg_left_rear, child link_upper_leg_left_rear, origin xyz=0 0 0 rpy=1.5707 0 0, axis 1 0 0, limit lower=-0.1963 upper=0.1963 effort=1000 velocity=100.0
- added joint joint_left_rear_3: type revolute, parent upper_leg_left_rear, child link_lower_leg_left_rear, origin xyz=0 0 0 rpy=0 1.5707 0, axis 1 0 0, limit lower=-1.64 upper=0.17 effort=1000 velocity=100.0
- added joint joint_left_rear_4: type revolute, parent lower_leg_left_rear, child link_foot_leg_left_rear, origin xyz=0 0 0 rpy=0 1.5707 0, axis 1 0 0, limit lower=-1.63 upper=0.62 effort=1000 velocity=100.0
- added joint joint_right_front_1: type revolute, parent base_link, child base_leg_right_front, origin xyz=0.23 -0.17 0.0 rpy=1.5707 0.785 0, axis 0 0 1, limit lower=0.21 upper=1.21 effort=1000 velocity=100.0
- added joint joint_right_front_2: type revolute, parent base_leg_right_front, child link_upper_leg_right_front, origin xyz=0 0 0 rpy=1.5707 0 0, axis 1 0 0, limit lower=-0.1963 upper=0.1963 effort=1000 velocity=100.0
- added joint joint_right_front_3: type revolute, parent upper_leg_right_front, child link_lower_leg_right_front, origin xyz=0 0 0 rpy=0 1.5707 0, axis 1 0 0, limit lower=-1.64 upper=0.17 effort=1000 velocity=100.0
- added joint joint_right_front_4: type revolute, parent lower_leg_right_front, child link_foot_leg_right_front, origin xyz=0 0 0 rpy=0 1.5707 0, axis 1 0 0, limit lower=-1.63 upper=0.62 effort=1000 velocity=100.0
- added joint joint_right_rear_1: type revolute, parent base_link, child base_leg_right_rear, origin xyz=-0.23 -0.17 0.0 rpy=1.5707 0.785 0, axis 0 0 1, limit lower=0.21 upper=1.21 effort=1000 velocity=100.0
- added joint joint_right_rear_2: type revolute, parent base_leg_right_rear, child link_upper_leg_right_rear, origin xyz=0 0 0 rpy=1.5707 0 0, axis 1 0 0, limit lower=-0.1963 upper=0.1963 effort=1000 velocity=100.0
- added joint joint_right_rear_3: type revolute, parent upper_leg_right_rear, child link_lower_leg_right_rear, origin xyz=0 0 0 rpy=0 1.5707 0, axis 1 0 0, limit lower=-1.64 upper=0.17 effort=1000 velocity=100.0
- added joint joint_right_rear_4: type revolute, parent lower_leg_right_rear, child link_foot_leg_right_rear, origin xyz=0 0 0 rpy=0 1.5707 0, axis 1 0 0, limit lower=-1.63 upper=0.62 effort=1000 velocity=100.0
- added joint lower_leg_left_front_joint: type fixed, parent link_lower_leg_left_front, child lower_leg_left_front, origin xyz=0 0 0.2 rpy=0 1.5707 0
- added joint lower_leg_left_rear_joint: type fixed, parent link_lower_leg_left_rear, child lower_leg_left_rear, origin xyz=0 0 0.2 rpy=0 1.5707 0
- added joint lower_leg_right_front_joint: type fixed, parent link_lower_leg_right_front, child lower_leg_right_front, origin xyz=0 0 0.2 rpy=0 1.5707 0
- added joint lower_leg_right_rear_joint: type fixed, parent link_lower_leg_right_rear, child lower_leg_right_rear, origin xyz=0 0 0.2 rpy=0 1.5707 0
- added joint upper_leg_left_front_joint: type fixed, parent link_upper_leg_left_front, child upper_leg_left_front, origin xyz=0 0 0.2 rpy=1.5707 0 0
- added joint upper_leg_left_rear_joint: type fixed, parent link_upper_leg_left_rear, child upper_leg_left_rear, origin xyz=0 0 0.2 rpy=1.5707 0 0
- added joint upper_leg_right_front_joint: type fixed, parent link_upper_leg_right_front, child upper_leg_right_front, origin xyz=0 0 0.2 rpy=1.5707 0 0
- added joint upper_leg_right_rear_joint: type fixed, parent link_upper_leg_right_rear, child upper_leg_right_rear, origin xyz=0 0 0.2 rpy=1.5707 0 0
